Commit message: robot model change by real

File: llb_nav/description/llb_car.urdf (robot description, URDF)
Before this commit: robot llb_car, 6 links, 5 joints
Joints:
- joint camera_link_to_base_link: origin xyz=0.13 0.0 0.13 rpy=0 0 0 -> xyz=0.02 0.0 0.206 rpy=0 0 0
- joint joint_base_wheel1: origin xyz=0.05 0.065 0.0 rpy=1.57 0 0 -> xyz=0.05 0.0975 0.0 rpy=1.57 0 0
- joint joint_base_wheel2: origin xyz=0.05 -0.065 0.0 rpy=1.57 0 0 -> xyz=0.05 -0.0975 0.0 rpy=1.57 0 0

File: llb_nav/description/llb_car.xacro (robot description, xacro)
@@ -7,7 +7,7 @@
   <xacro:property name="body_pos" value="0 0 0.05" />
   <xacro:property name="wheel_radius" value="0.032" />
-  <xacro:property name="wheel_length" value="0.02" />
-  <xacro:property name="wheel1_pos" value="0.05 0.065 0.0" />
-  <xacro:property name="wheel2_pos" value="0.05 -0.065 0.0" />
+  <xacro:property name="wheel_length" value="0.027" />
+  <xacro:property name="wheel1_pos" value="0.05 0.0975 0.0" />
+  <xacro:property name="wheel2_pos" value="0.05 -0.0975 0.0" />
   <xacro:macro name="wheel" params="wheelname position">
     <link name="${wheelname}">
@@ -53,5 +53,5 @@
 		<parent link="base_link" />
 		<child link="camera_link" />
-		<origin rpy="0 0 0" xyz="0.13 0.0 0.13" />
+		<origin rpy="0 0 0" xyz="0.02 0.0 0.206" />
 	</joint>
 	<link name="camera_depth_frame">

Commit message: add udev rules for arduinos serial port remap

File: llb_nav/description/llb_car.urdf (robot description, URDF)
Before this commit: robot llb_car, 6 links, 5 joints
Links:
- added link base_laser_bottom, mass 0.1; collision box size=0.05 0.05 0.041; visual box size=0.05 0.05 0.041
- added link base_laser_middle, mass 0.1; collision cylinder length=0.0115 radius=.02; visual cylinder length=0.0115 radius=.02
- added link laser, mass 0.1; collision cylinder length=0.0175 radius=.0185; visual cylinder length=0.0175 radius=.0185
- link base_link: geometry visual box size=.2 .12 .11
- link wheel1: geometry visual cylinder length=0.055 radius=0.0575
- link wheel2: geometry visual cylinder length=0.055 radius=0.0575
Joints:
- added joint base_laser_bottom_joint: type fixed, parent base_link, child base_laser_bottom, origin xyz=0.0 0.0 0.1305 rpy=0 0 0 
- added joint base_laser_joint: type fixed, parent base_laser_middle, child laser, origin xyz=0 0 0.0145 rpy=0 0 0
- added joint base_laser_middle_joint: type fixed, parent base_laser_bottom, child base_laser_middle, origin xyz=0 0 0.02625 rpy=0 0 0
- joint camera_link_to_base_link: origin xyz=0.02 0.0 0.206 rpy=0 0 0 -> xyz=0.04 0.0 0.12 rpy=0 0 0
