Commit message: align

File: llb_nav/description/higherRplidar_camera_car.urdf (robot description, URDF)
Before this commit: robot auto_pro1, 11 links, 10 joints
Links:
- removed link camera_depth_frame
- removed link camera_depth_optical_frame
- removed link camera_link
Joints:
- removed joint camera_depth_joint
- removed joint camera_link_to_base_link
- removed joint depth_optical_joint

Commit message: change autolabor device model

File: llb_nav/description/higherRplidar_camera_car.urdf (robot description, URDF)
Before this commit: robot auto_pro1, 8 links, 7 joints
Links:
- removed link base_l1_wheel_link
- removed link base_l2_wheel_link
- removed link base_laser_bottom
- removed link base_laser_middle
- removed link base_link
- removed link base_r1_wheel_link
- removed link base_r2_wheel_link
- removed link laser
- added link robot1/base_l1_wheel_link; visual cylinder length=0.054 radius=0.058
- added link robot1/base_l2_wheel_link; visual cylinder length=0.054 radius=0.058
- added link robot1/base_laser_bottom, mass 0.1; collision box size=0.05 0.05 0.041; visual box size=0.05 0.05 0.041
- added link robot1/base_laser_middle, mass 0.1; collision cylinder length=0.0115 radius=.02; visual cylinder length=0.0115 radius=.02
- added link robot1/base_link; collision box size=0.726 0.615 0.2; visual box size=0.354 0.181 0.11
- added link robot1/base_r1_wheel_link; visual cylinder length=0.054 radius=0.058
- added link robot1/base_r2_wheel_link; visual cylinder length=0.054 radius=0.058
- added link robot1/laser, mass 0.1; collision cylinder length=0.0175 radius=.0185; visual cylinder length=0.0175 radius=.0185
Joints:
- removed joint base_l1_wheel_joint
- removed joint base_l2_wheel_joint
- removed joint base_laser_bottom_joint
- removed joint base_laser_joint
- removed joint base_laser_middle_joint
- removed joint base_r1_wheel_joint
- removed joint base_r2_wheel_joint
- added joint robot1/base_l1_wheel_joint: type fixed, parent robot1/base_link, child robot1/base_l1_wheel_link, origin xyz=0.119 0.1275 -0.065 rpy=1.57075 0 0 , axis 0 0 1, limit effort=100 velocity=100
- added joint robot1/base_l2_wheel_joint: type fixed, parent robot1/base_link, child robot1/base_l2_wheel_link, origin xyz=-0.119 0.1275 -0.065 rpy=1.57075 0 0 , axis 0 0 1, limit effort=100 velocity=100
- added joint robot1/base_laser_bottom_joint: type fixed, parent robot1/base_link, child robot1/base_laser_bottom, origin xyz=0.0 0.0 0.091 rpy=0 0 0 
- added joint robot1/base_laser_joint: type fixed, parent robot1/base_laser_middle, child robot1/laser, origin xyz=0 0 0.0145 rpy=0 0 0
- added joint robot1/base_laser_middle_joint: type fixed, parent robot1/base_laser_bottom, child robot1/base_laser_middle, origin xyz=0 0 0.02625 rpy=0 0 0
- added joint robot1/base_r1_wheel_joint: type fixed, parent robot1/base_link, child robot1/base_r1_wheel_link, origin xyz=0.119 -0.1275 -0.065 rpy=-1.57075 0 0 , axis 0 0 1, limit effort=100 velocity=100
- added joint robot1/base_r2_wheel_joint: type fixed, parent robot1/base_link, child robot1/base_r2_wheel_link, origin xyz=-0.119 -0.1275 -0.065 rpy=-1.57075 0 0 , axis 0 0 1, limit effort=100 velocity=100

Commit message: base

File: llb_nav/description/higherRplidar_camera_car.urdf (robot description, URDF)
Before this commit: robot robot1/auto_pro1, 8 links, 7 joints
Links:
- removed link robot1/base_l1_wheel_link
- removed link robot1/base_l2_wheel_link
- removed link robot1/base_laser_bottom
- removed link robot1/base_laser_middle
- removed link robot1/base_link
- removed link robot1/base_r1_wheel_link
- removed link robot1/base_r2_wheel_link
- removed link robot1/laser
- added link base_l1_wheel_link; visual cylinder length=0.054 radius=0.058
- added link base_l2_wheel_link; visual cylinder length=0.054 radius=0.058
- added link base_laser_bottom, mass 0.1; collision box size=0.05 0.05 0.041; visual box size=0.05 0.05 0.041
- added link base_laser_middle, mass 0.1; collision cylinder length=0.0115 radius=.02; visual cylinder length=0.0115 radius=.02
- added link base_link; collision box size=0.726 0.615 0.2; visual box size=0.354 0.181 0.11
- added link base_r1_wheel_link; visual cylinder length=0.054 radius=0.058
- added link base_r2_wheel_link; visual cylinder length=0.054 radius=0.058
- added link laser, mass 0.1; collision cylinder length=0.0175 radius=.0185; visual cylinder length=0.0175 radius=.0185
Joints:
- removed joint robot1/base_l1_wheel_joint
- removed joint robot1/base_l2_wheel_joint
- removed joint robot1/base_laser_bottom_joint
- removed joint robot1/base_laser_joint
- removed joint robot1/base_laser_middle_joint
- removed joint robot1/base_r1_wheel_joint
- removed joint robot1/base_r2_wheel_joint
- added joint base_l1_wheel_joint: type fixed, parent base_link, child base_l1_wheel_link, origin xyz=0.119 0.1275 -0.065 rpy=1.57075 0 0 , axis 0 0 1, limit effort=100 velocity=100
- added joint base_l2_wheel_joint: type fixed, parent base_link, child base_l2_wheel_link, origin xyz=-0.119 0.1275 -0.065 rpy=1.57075 0 0 , axis 0 0 1, limit effort=100 velocity=100
- added joint base_laser_bottom_joint: type fixed, parent base_link, child base_laser_bottom, origin xyz=0.0 0.0 0.091 rpy=0 0 0 
- added joint base_laser_joint: type fixed, parent base_laser_middle, child laser, origin xyz=0 0 0.0145 rpy=0 0 0
- added joint base_laser_middle_joint: type fixed, parent base_laser_bottom, child base_laser_middle, origin xyz=0 0 0.02625 rpy=0 0 0
- added joint base_r1_wheel_joint: type fixed, parent base_link, child base_r1_wheel_link, origin xyz=0.119 -0.1275 -0.065 rpy=-1.57075 0 0 , axis 0 0 1, limit effort=100 velocity=100
- added joint base_r2_wheel_joint: type fixed, parent base_link, child base_r2_wheel_link, origin xyz=-0.119 -0.1275 -0.065 rpy=-1.57075 0 0 , axis 0 0 1, limit effort=100 velocity=100
